File: 02_Assemble/gl65.kicad_pcb (KiCad board)
At the start: 2 copper layers, 304.4 x 98.8 mm, 137 parts, among them J1 Conn_01x02, SW1 SW_PUSH, SW10 SW_PUSH, SW11 SW_PUSH, SW12 SW_PUSH, SW13 SW_PUSH, SW14 SW_PUSH, SW15 SW_PUSH, SW16 SW_PUSH, SW17 SW_PUSH, SW18 SW_PUSH, SW19 SW_PUSH, SW2 SW_PUSH, SW20 SW_PUSH, SW21 SW_PUSH, SW22 SW_PUSH, SW23 SW_PUSH, SW24 SW_PUSH, SW25 SW_PUSH, SW26 SW_PUSH, SW27 SW_PUSH, SW28 SW_PUSH, SW29 SW_PUSH, SW3 SW_PUSH, SW30 SW_PUSH, SW31 SW_PUSH, SW32 SW_PUSH, SW33 SW_PUSH, SW34 SW_PUSH, SW35 SW_PUSH, SW36 SW_PUSH, SW37 SW_PUSH, SW38 SW_PUSH, SW39 SW_PUSH, SW4 SW_PUSH, SW40 SW_PUSH, SW41 SW_PUSH, SW42 SW_PUSH, SW43 SW_PUSH, SW44 SW_PUSH, SW45 SW_PUSH, SW46 SW_PUSH, SW47 SW_PUSH, SW48 SW_PUSH, SW49 SW_PUSH, SW5 SW_PUSH, SW50 SW_PUSH, SW51 SW_PUSH, SW52 SW_PUSH, SW53 SW_PUSH, SW54 SW_PUSH, SW55 SW_PUSH, SW56 SW_PUSH, SW57 SW_PUSH, SW58 SW_PUSH, SW59 SW_PUSH, SW6 SW_PUSH, SW60 SW_PUSH, SW61 SW_PUSH, SW62 SW_PUSH, SW63 SW_PUSH, SW64 SW_PUSH, SW65 SW_PUSH, SW66 SW_PUSH, SW67 SW_PUSH, SW68 SW_PUSH, SW7 SW_PUSH, SW8 SW_PUSH, SW9 SW_PUSH, U1 BLEMicroPro

Commit message: サリチル酸さんのレビューの指摘を修正。 ・ProMicroの位置を0.3mm下げる ・ResetスイッチをProMicroのすぐ横に移動 ・ソケットのパッドにビアを打たないように変更 ・ダイオードの向きを統一 ・2U以上のキーのリファレンスを表示
Parts:
- moved SW68 48.5 mm to (61.5, 19.5)
- moved D52 3.72 mm to (192.7, 94.2), turned to 90 degrees
- moved D54 3.72 mm to (230.8, 94.2), turned to 90 degrees
- moved D53 3.71 mm to (211.8, 94.2), turned to 90 degrees
- moved U1 0.30 mm to (34.5, 28.2)
- turned D10 to 90 degrees
- turned D11 to 90 degrees
- turned D12 to 90 degrees
- turned D13 to 90 degrees
- turned D14 to 90 degrees
- turned D15 to 90 degrees
- turned D23 to 90 degrees
- turned D24 to 90 degrees
- turned D25 to 90 degrees
- turned D26 to 90 degrees
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Routing:
- net Row0: track 301.3 -> 367.9 mm
- net Row1: track 323.0 -> 389.5 mm
- net Row4: track 396.0 -> 451.9 mm
- net Row3: track 376.2 -> 429.6 mm
- net Row2: track 360.8 -> 409.5 mm
- net GND: track 189.5 -> 158.9 mm, vias 4 -> 2
- net Col6: track 408.6 -> 397.4 mm, vias 9 -> 13
- net Net-(D52-Pad1): track 8.71 -> 19.5 mm, vias 0 -> 2
- net Net-(D54-Pad1): track 8.71 -> 19.0 mm, vias 0 -> 2
- net Net-(D53-Pad1): track 8.71 -> 18.7 mm, vias 0 -> 2
- net Net-(D26-Pad1): track 8.71 -> 16.7 mm
- net Net-(D27-Pad1): track 8.71 -> 16.3 mm
- net Net-(D28-Pad1): track 8.71 -> 16.3 mm
- net Net-(D13-Pad1): track 8.71 -> 16.2 mm
- net Net-(D38-Pad1): track 8.71 -> 16.1 mm
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